File: activeload_ctrl_hardware/stm32f030f4p6/stm32f030f4p6.kicad_pcb (KiCad board)
At the start: 2 copper layers, 98 x 85 mm, 44 parts, among them J1 Supply, J2 LCD, J3 SWD, J4 USART, J5 Module, J6 Supply, SW2 SW_Push, SW3 SW_Push, SW4 SW_Push, U1 STM32F030F4Px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

Commit message: PCB processed
Parts:
- moved R7 152.1 mm to (258.0, 71.0)
- moved C3 141.7 mm to (241.2, 86.5)
- moved C4 141.7 mm to (241.2, 89.5)
- moved C1 138.9 mm to (228.0, 93.8)
- moved R8 135.6 mm to (241.2, 77.5)
- moved R9 135.6 mm to (241.2, 80.8)
- moved R6 131.1 mm to (233.6, 89.5), turned to 180 degrees
- moved C11 124.4 mm to (223.2, 93.8), turned to 180 degrees
- moved R11 123.3 mm to (233.4, 80.5)
- moved R12 123.3 mm to (233.4, 83.8)
- moved R3 115.6 mm to (214.4, 82.9)
- moved R4 115.6 mm to (214.4, 86.2)
- moved R5 115.6 mm to (214.4, 89.5)
- moved R13 94.3 mm to (203.9, 86.2), turned to 180 degrees
- moved R14 94.3 mm to (203.9, 89.5), turned to 180 degrees
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Routing:
- net +12V: track 0.00 -> 49.0 mm
- net GND: track 0.00 -> 46.3 mm
- net +3.3V: track 0.00 -> 25.4 mm
- net +5V: track 0.00 -> 18.2 mm
- net /BTN3: track 0.00 -> 17.4 mm
- net /I2C_SCL: track 0.00 -> 12.6 mm
- net /BTN2: track 0.00 -> 12.5 mm
- net /BTN1: track 0.00 -> 12.5 mm
- net +3.3VADC: track 0.00 -> 11.5 mm
- net /I2C_SDA: track 0.00 -> 9.50 mm

Commit message: PCB in grogress
Parts:
- added C12: 0.1u, Capacitor_SMD:C_0805_2012Metric_Pad1.18x1.45mm_HandSolder, F.Cu at (183.5, 93.5)
- moved C6 25.6 mm to (167.0, 93.5), turned to 180 degrees
- moved C10 15.8 mm to (173.0, 83.0), turned to 180 degrees
- moved C7 9.86 mm to (157.5, 85.5), turned to -90 degrees
- moved C9 9.80 mm to (174.0, 85.5)
- moved C8 8.45 mm to (156.5, 83.0), turned to 180 degrees
- moved U4 7.02 mm to (181.3, 87.3), turned to 180 degrees
- moved U3 5.37 mm to (164.8, 87.5), turned to 180 degrees
- moved R6 1.75 mm to (233.6, 91.2)
Routing:
- net Net-(D3-A): track 0.00 -> 64.2 mm
- net Net-(D1-A): track 0.00 -> 58.5 mm
- net Net-(D2-A): track 0.00 -> 52.7 mm
- net +5V: track 18.2 -> 25.7 mm
- net +3.3V: track 25.4 -> 32.8 mm
- net /BTN3: track 17.4 -> 15.8 mm
