File: activeload_ctrl_hardware/stm32f030f4p6/stm32f030f4p6.kicad_sch (KiCad schematic)
At the start: 43 parts

Commit message: PCB start
Parts:
- removed C? (x2): 100u, Capacitor_THT:CP_Radial_D4.0mm_P2.00mm, symbol Device:CP
- removed C?: 470u 25v, Capacitor_THT:C_Radial_D8.0mm_H7.0mm_P3.50mm, symbol Device:CP
- removed R?: 10k, Resistor_SMD:R_1206_3216Metric_Pad1.30x1.75mm_HandSolder, symbol Device:R
- removed RN? (x4): 10k, Resistor_SMD:R_Array_Convex_4x1206, symbol Device:R_Pack04_Split
- removed SW?: (no value), Rotary_Encoder:RotaryEncoder_Alps_EC12E-Switch_Vertical_H20mm, symbol Device:Rotary_Encoder_Switch
- removed U?: AMS1117-5.0, Package_TO_SOT_SMD:SOT-223-3_TabPin2, symbol Regulator_Linear:AMS1117-5.0
- removed U?: AMS1117-3.3, Package_TO_SOT_SMD:SOT-223-3_TabPin2, symbol Regulator_Linear:AMS1117-3.3
- added C5: 470u, Capacitor_THT:C_Radial_D8.0mm_H7.0mm_P3.50mm, symbol Device:C_Polarized
- added C7, C9: 100u, Capacitor_THT:CP_Radial_D4.0mm_P2.00mm, symbol Device:C_Polarized
- added J4: USART, Connector_PinHeader_2.54mm:PinHeader_1x03_P2.54mm_Vertical, symbol Connector_Generic:Conn_01x03
- added R1, R2, R3, R4, R5: 10k, Resistor_SMD:R_1206_3216Metric_Pad1.30x1.75mm_HandSolder, symbol Device:R
- added SW1: ~, Rotary_Encoder:RotaryEncoder_Alps_EC12E-Switch_Vertical_H20mm, symbol Device:RotaryEncoder_Switch
- added U3: AMS1117-5.0, Package_TO_SOT_SMD:SOT-223-3_TabPin2, symbol Regulator_Linear:AMS1117-5.0
- added U4: AMS1117-3.3, Package_TO_SOT_SMD:SOT-223-3_TabPin2, symbol Regulator_Linear:AMS1117-3.3
- gave numbers to parts that had none: 32
Connections:
- net LED_G is gone; now on net SWDIO: R13.1
- net LED_R is gone; now on net SWCLK: R14.1
- net +5V: now also C7.1, U3.2 (VO)
- net BTN1: now also U1.7 (PA1), R4.2
- net BTN2: now also U1.10 (PA4), R5.2
- net BTN3: now also U1.11 (PA5)
- net ENC_BTN: now also U1.6 (PA0), R3.2, SW1.S1
- net GND: now also C5.2, C7.2, C9.2, J4.3 (Pin_3), SW1.C, SW1.S2, U3.1 (GND), U4.1 (GND)
- net LED_Y: now also U1.2 (PF0)
- net USART_RX: now also J4.2 (Pin_2)
- net USART_TX: now also J4.1 (Pin_1)
- net WOE: now also U1.14 (PB1)
- net ~{WOE}: now also U1.3 (PF1)
- net at R8.1: now also R1.2, SW1.A
- net at R9.1: now also R2.2, SW1.B
- net +3V3 renamed +3.3V
- net +3.3V: now also C9.1, R1.1, R2.1, R3.1, R4.1, R5.1, U4.2 (VO)
- net +VPS renamed +12V
- net +12V: now also C5.1, U3.3 (VI), U4.3 (VI)
Other:
- note added: "Control elements"
- note added: "Indication"
- note added: "MCU&EEPROM"
- note added: "Output connection"
- moved on the sheet: C1, C10, C11, C2, C3, C4, C6, C8, D1, D2, D3, J1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

Commit message: PCB in grogress
Parts:
- added C12: 0.1u, Capacitor_SMD:C_0805_2012Metric_Pad1.18x1.45mm_HandSolder, symbol Device:C
Connections:
- net +12V: now also C12.1
- net GND: now also C12.2
Other:
- moved on the sheet: C5, J1
Changed lines of the file:
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@@
 	)
 	(junction
-		(at 58.42 142.24)
+		(at 52.07 142.24)
 		(diameter 0)
 		(color 0 0 0 0)
@@
 	)
 	(junction
-		(at 58.42 129.54)
+		(at 63.5 129.54)
+		(diameter 0)
+		(color 0 0 0 0)
+	)
+	(junction
+		(at 63.5 142.24)
+		(diameter 0)
+		(color 0 0 0 0)
+	)
+	(junction
+		(at 52.07 129.54)
 		(diameter 0)
 		(color 0 0 0 0)
@@
 	(wire
 		(pts
-			(xy 50.8 129.54) (xy 58.42 129.54)
+			(xy 44.45 129.54) (xy 52.07 129.54)
 		)
 		(stroke
@@
 	(wire
 		(pts
-			(xy 73.66 142.24) (xy 58.42 142.24)
+			(xy 73.66 142.24) (xy 63.5 142.24)
 		)
 		(stroke
@@
 	(wire
 		(pts
-			(xy 53.34 142.24) (xy 58.42 142.24)
+			(xy 46.99 142.24) (xy 52.07 142.24)
 		)
 		(stroke
@@
 	(wire
 		(pts
-			(xy 50.8 134.62) (xy 53.34 134.62)
+			(xy 44.45 134.62) (xy 46.99 134.62)
+		)
+		(stroke
+			(width 0)
+			(type default)
+		)
+	)
+	(wire
+		(pts
+			(xy 63.5 129.54) (xy 73.66 129.54)
 		)
 		(stroke
@@
 	(wire
 		(pts
+			(xy 63.5 129.54) (xy 63.5 132.08)
+		)
+		(stroke
+			(width 0)
+			(type default)
+		)
+	)
+	(wire
+		(pts
 			(xy 198.12 67.31) (xy 198.12 68.58)
 		)
@@
 	(wire
 		(pts
-			(xy 58.42 129.54) (xy 58.42 132.08)
+			(xy 52.07 129.54) (xy 52.07 132.08)
 		)
 		(stroke
@@
 	(wire
 		(pts
-			(xy 58.42 139.7) (xy 58.42 142.24)
+			(xy 52.07 139.7) (xy 52.07 142.24)
 		)
 		(stroke
@@
 	(wire
 		(pts
-			(xy 58.42 129.54) (xy 73.66 129.54)
+			(xy 52.07 129.54) (xy 63.5 129.54)
 		)
 		(stroke
@@
 	(wire
 		(pts
-			(xy 58.42 128.27) (xy 58.42 129.54)
+			(xy 52.07 128.27) (xy 52.07 129.54)
 		)
 		(stroke
@@
 	(wire
 		(pts
+			(xy 63.5 142.24) (xy 52.07 142.24)
+		)
+		(stroke
+			(width 0)
+			(type default)
+		)
+	)
+	(wire
+		(pts
 			(xy 115.57 142.24) (xy 115.57 139.7)
 		)
@@
 	(wire
 		(pts
-			(xy 53.34 134.62) (xy 53.34 142.24)
+			(xy 46.99 134.62) (xy 46.99 142.24)
 		)
 		(stroke
@@
 	(wire
 		(pts
+			(xy 63.5 139.7) (xy 63.5 142.24)
+		)
+		(stroke
+			(width 0)
+			(type default)
+		)
+	)
+	(wire
+		(pts
 			(xy 187.96 43.18) (xy 187.96 46.99)
 		)
@@
 	)
 	(symbol
+		(lib_id "Device:C")
+		(at 63.5 135.89 0)
+		(unit 1)
+		(exclude_from_sim no)
+		(in_bom yes)
+		(on_board yes)
+		(dnp no)
+		(property "Reference" "C12"
+			(at 66.421 134.7216 0)
+			(effects
+				(font
+					(size 1.27 1.27)
+				)
+				(justify left)
+			)
+		)
+		(property "Value" "0.1u"
+			(at 66.421 137.033 0)
+			(effects
+				(font
+					(size 1.27 1.27)
+				)
+				(justify left)
+			)
+		)
+		(property "Footprint" "Capacitor_SMD:C_0805_2012Metric_Pad1.18x1.45mm_HandSolder"
+			(at 64.4652 139.7 0)
+			(effects
+				(font
+					(size 1.27 1.27)
+				)
+				(hide yes)
+			)
+		)
+		(property "Datasheet" "~"
+			(at 63.5 135.89 0)
+			(effects
+				(font
+					(size 1.27 1.27)
+				)
+				(hide yes)
+			)
+		)
+		(property "Description" ""
+			(at 63.5 135.89 0)
+			(effects
+				(font
+					(size 1.27 1.27)
+				)
+				(hide yes)
+			)
+		)
+		(pin "1"
+		)
+		(pin "2"
+		)
+		(instances
+			(project "stm32f030f4p6"
+				(path "/d7d9441b-f478-4590-87f0-c9f097cf72ee"
+					(reference "C12")
+					(unit 1)
+				)
+			)
+		)
+	)
+	(symbol
 		(lib_id "Device:R")
 		(at 223.52 119.38 270)
@@
 	(symbol
 		(lib_id "power:+12V")
-		(at 58.42 128.27 0)
+		(at 52.07 128.27 0)
 		(unit 1)
 		(exclude_from_sim no)
@@
 		(fields_autoplaced yes)
 		(property "Reference" "#PWR010"
-			(at 58.42 132.08 0)
+			(at 52.07 132.08 0)
 			(effects
 				(font
@@
 		)
 		(property "Value" "+12V"
-			(at 58.42 124.1369 0)
+			(at 52.07 124.1369 0)
 			(effects
 				(font
@@
 		)
 		(property "Footprint" ""
-			(at 58.42 128.27 0)
+			(at 52.07 128.27 0)
 			(effects
 				(font
@@
 		)
 		(property "Datasheet" ""
-			(at 58.42 128.27 0)
+			(at 52.07 128.27 0)
 			(effects
 				(font
@@
 		)
 		(property "Description" "Power symbol creates a global label with name \"+12V\""
-			(at 58.42 128.27 0)
+			(at 52.07 128.27 0)
 			(effects
 				(font
@@
 	(symbol
 		(lib_id "Connector:Barrel_Jack")
-		(at 43.18 132.08 0)
+		(at 36.83 132.08 0)
 		(unit 1)
 		(exclude_from_sim no)
@@
 		(fields_autoplaced yes)
 		(property "Reference" "J1"
-			(at 43.18 124.3035 0)
+			(at 36.83 124.3035 0)
 			(effects
 				(font
@@
 		)
 		(property "Value" "Supply"
-			(at 43.18 127.0786 0)
+			(at 36.83 127.0786 0)
 			(effects
 				(font
@@
 		)
 		(property "Footprint" "Connector_BarrelJack:BarrelJack_Horizontal"
-			(at 44.45 133.096 0)
+			(at 38.1 133.096 0)
 			(effects
 				(font
@@
 		)
 		(property "Datasheet" "~"
-			(at 44.45 133.096 0)
+			(at 38.1 133.096 0)
 			(effects
 				(font
@@
 		)
 		(property "Description" ""
-			(at 43.18 132.08 0)
+			(at 36.83 132.08 0)
 			(effects
 				(font
@@
 	(symbol
 		(lib_id "Device:C_Polarized")
-		(at 58.42 135.89 0)
+		(at 52.07 135.89 0)
 		(unit 1)
 		(exclude_from_sim no)
@@
 		(dnp no)
 		(property "Reference" "C5"
-			(at 61.341 133.7888 0)
+			(at 54.991 133.7888 0)
 			(effects
 				(font
@@
 		)
 		(property "Value" "470u"
-			(at 61.341 136.2131 0)
+			(at 54.991 136.2131 0)
 			(effects
 				(font
@@
 		)
 		(property "Footprint" "Capacitor_THT:C_Radial_D8.0mm_H7.0mm_P3.50mm"
-			(at 59.3852 139.7 0)
+			(at 53.0352 139.7 0)
 			(effects
 				(font
@@
 		)
 		(property "Datasheet" "~"
-			(at 58.42 135.89 0)
+			(at 52.07 135.89 0)
 			(effects
 				(font
@@
 		)
 		(property "Description" "Polarized capacitor"
-			(at 58.42 135.89 0)
+			(at 52.07 135.89 0)
 			(effects
 				(font
@@
 		)
 		(property "Voltage" "25v"
-			(at 63.246 138.176 0)
+			(at 56.896 138.176 0)
 			(effects
 				(font
