File: activeload_ctrl_hardware/stm32f030k6t6/stm32f030k6t6.kicad_pcb (KiCad board)
At the start: 2 copper layers, 98 x 85 mm, 46 parts, among them J1 Supply, J2 LCD, J3 SWD, J4 USART, J5 Module, J6 Supply, SW2 SW_Push, SW3 SW_Push, SW4 SW_Push, U1 STM32F030K6Tx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

Commit message: stm32f030k6t6  add testpoint to scheme
Parts:
- added TP1: TestPoint, Connector_PinHeader_2.54mm:PinHeader_1x01_P2.54mm_Vertical, F.Cu at (240.0, 73.9)
- added TP2: TestPoint, Connector_PinHeader_2.54mm:PinHeader_1x01_P2.54mm_Vertical, F.Cu at (240.0, 68.9)
- added TP3: TestPoint, Connector_PinHeader_2.54mm:PinHeader_1x01_P2.54mm_Vertical, F.Cu at (240.0, 63.9)
Connections:
- U1 pad 6: unconnected-(U1-PA0-Pad6) -> Net-(U1-PA0)
- U1 pad 7: unconnected-(U1-PA1-Pad7) -> Net-(U1-PA1)
Routing:
- net Net-(U1-PA0): track 0.00 -> 34.1 mm
- net Net-(U1-PA1): track 0.00 -> 34.1 mm
- net Net-(R2-Pad2): track 61.7 -> 65.7 mm
- net Net-(R1-Pad2): track 53.7 -> 57.4 mm
- net /ENC_BTN: track 86.4 -> 89.0 mm
- net GND: track 211.8 -> 210.2 mm
- net /I2C_SDA: track 93.4 -> 92.7 mm
- net +3.3V: vias 4 -> 6

Commit message: stm32f030k6t6 add logo to pcb
Parts:
- added G***: LOGO, UVM_Logo:bel_fire_small, F.Cu at (235.2, 87.6)
- added G***: LOGO, UVM_Logo:UVM_small, F.Cu at (235.7, 97.9)
Other:
- outline, holes or cut-outs redrawn
- board text added: "Ruthenia Alba 2024"
